Commit message: Simulation configuration

File: xarm1s_moveit_config/config/xarm_1s.ros2_control.xacro (robot description, xacro)
@@ -1,10 +1,20 @@
 <?xml version="1.0"?>
 <robot xmlns:xacro="http://www.ros.org/wiki/xacro">
-    <xacro:macro name="xarm_1s_ros2_control" params="name initial_positions_file">
-        <xacro:property name="initial_positions" value="${load_yaml(initial_positions_file)['initial_positions']}"/>
+    <xacro:macro name="xarm_1s_ros2_control" params="name initial_positions_file is_simulation">
+        <xacro:property name="initial_positions" value="${xacro.load_yaml(initial_positions_file)['initial_positions']}"/>
+        <gazebo>
+          <plugin filename="libgz_ros2_control-system.so" name="gz_ros2_control::GazeboSimROS2ControlPlugin">
+            <parameters>$(find xarm1s_moveit_config)/config/ros2_controllers.yaml</parameters>
+          </plugin>
+        </gazebo>
         <ros2_control name="${name}" type="system">
             <hardware>
                 <!-- By default, set up controllers for simulation. This won't work on real hardware -->
-                <plugin>mock_components/GenericSystem</plugin>
+                <xacro:if value="${is_simulation}">
+                  <plugin>gz_ros2_control/GazeboSimSystem</plugin>
+                </xacro:if>
+                <xacro:unless value="${is_simulation}">
+                  <plugin>mock_components/GenericSystem</plugin>
+                </xacro:unless>
             </hardware>
             <joint name="arm6">
@@ -50,4 +60,8 @@
                 <state_interface name="velocity"/>
             </joint>
+            <joint name="arm1_left">
+                <state_interface name="position"/>
+                <state_interface name="velocity"/>
+            </joint>
         </ros2_control>
     </xacro:macro>

File: xarm1s_moveit_config/config/xarm_1s.urdf.xacro (robot description, xacro)
@@ -2,8 +2,14 @@
 <robot xmlns:xacro="http://www.ros.org/wiki/xacro" name="xarm_1s">
     <xacro:arg name="initial_positions_file" default="initial_positions.yaml" />
+    <xacro:arg name="is_simulation" default="false" />
     <!-- Import xarm_1s urdf file -->
     <xacro:include filename="$(find xarm_description)/urdf/xarm_1s.urdf.xacro" />
     <!-- Import control_xacro -->
     <xacro:include filename="xarm_1s.ros2_control.xacro" />
-    <xacro:xarm_1s_ros2_control name="FakeSystem" initial_positions_file="$(arg initial_positions_file)"/>
+    <xacro:if value="$(arg is_simulation)">
+        <xacro:xarm_1s_ros2_control name="GazeboSimSystem" initial_positions_file="$(arg initial_positions_file)" is_simulation="$(arg is_simulation)"/>
+    </xacro:if>
+    <xacro:unless value="$(arg is_simulation)">
+        <xacro:xarm_1s_ros2_control name="FakeSystem" initial_positions_file="$(arg initial_positions_file)" is_simulation="$(arg is_simulation)"/>
+    </xacro:unless>
 </robot>

File: xarm_description/urdf/xarm_1s.urdf.xacro (robot description, xacro)
@@ -17,6 +17,6 @@
       <origin rpy="0 0 0" xyz="0.0 0.0 0.0" />
       <geometry>
-        <!-- <mesh filename="package://xarm_1s_description/meshes/base.stl" scale="1.0 1.0 1.0" /> -->
-        <mesh filename="file://$(find xarm_description)/meshes/base.stl" scale="1.0 1.0 1.0" />
+        <mesh filename="package://xarm_1s_description/meshes/base.stl" scale="1.0 1.0 1.0" />
+        <!-- <mesh filename="file://$(find xarm_description)/meshes/base.stl" scale="1.0 1.0 1.0" /> -->
       </geometry>
       <material name="blue" />
@@ -53,4 +53,8 @@
       </geometry>
     </collision>
+    <inertial>
+      <mass value="1"/>
+      <inertia ixx="0.4" ixy="0.0" ixz="0.0" iyy="0.4" iyz="0.0" izz="0.2"/>
+    </inertial>
   </link>
   <joint name="arm5" type="revolute">

Commit message: planning pipeline config files

File: xarm1s_moveit_config/config/xarm_1s.ros2_control.xacro (robot description, xacro)
@@ -19,5 +19,8 @@
             </hardware>
             <joint name="arm6">
-                <command_interface name="position"/>
+                <command_interface name="position">
+                  <param name="min">-2.09439435</param>
+                  <param name="max">2.09439435</param>
+                </command_interface>
                 <state_interface name="position">
                   <param name="initial_value">${initial_positions['arm6']}</param>
@@ -26,5 +29,8 @@
             </joint>
             <joint name="arm5">
-                <command_interface name="position"/>
+                <command_interface name="position">
+                  <param name="min">-2.09439435</param>
+                  <param name="max">2.09439435</param>
+                </command_interface>
                 <state_interface name="position">
                   <param name="initial_value">${initial_positions['arm5']}</param>
@@ -33,5 +39,8 @@
             </joint>
             <joint name="arm4">
-                <command_interface name="position"/>
+                <command_interface name="position">
+                  <param name="min">-2.09439435</param>
+                  <param name="max">2.09439435</param>
+                </command_interface>
                 <state_interface name="position">
                   <param name="initial_value">${initial_positions['arm4']}</param>
@@ -40,5 +49,8 @@
             </joint>
             <joint name="arm3">
-                <command_interface name="position"/>
+                <command_interface name="position">
+                  <param name="min">-2.09439435</param>
+                  <param name="max">2.09439435</param>
+                </command_interface>
                 <state_interface name="position">
                   <param name="initial_value">${initial_positions['arm3']}</param>
@@ -47,5 +59,8 @@
             </joint>
             <joint name="arm2">
-                <command_interface name="position"/>
+                <command_interface name="position">
+                  <param name="min">-2.09439435</param>
+                  <param name="max">2.09439435</param>
+                </command_interface>
                 <state_interface name="position">
                   <param name="initial_value">${initial_positions['arm2']}</param>
@@ -54,5 +69,8 @@
             </joint>
             <joint name="arm1">
-                <command_interface name="position"/>
+                <command_interface name="position">
+                  <param name="min">0</param>
+                  <param name="max">0.8464847</param>
+                </command_interface>
                 <state_interface name="position">
                   <param name="initial_value">${initial_positions['arm1']}</param>

File: xarm_description/urdf/xarm_1s.urdf.xacro (robot description, xacro)
@@ -17,6 +17,6 @@
       <origin rpy="0 0 0" xyz="0.0 0.0 0.0" />
       <geometry>
-        <mesh filename="package://xarm_1s_description/meshes/base.stl" scale="1.0 1.0 1.0" />
-        <!-- <mesh filename="file://$(find xarm_description)/meshes/base.stl" scale="1.0 1.0 1.0" /> -->
+        <!-- <mesh filename="package://xarm_1s_description/meshes/base.stl" scale="1.0 1.0 1.0" /> -->
+        <mesh filename="file://$(find xarm_description)/meshes/base.stl" scale="1.0 1.0 1.0" />
       </geometry>
       <material name="blue" />
@@ -29,4 +29,8 @@
       </geometry>
     </collision>
+    <inertial>
+      <mass value="0.1"/>
+      <inertia ixx="0.4" ixy="0.0" ixz="0.0" iyy="0.4" iyz="0.0" izz="0.2"/>
+    </inertial>
   </link>
   <joint name="arm6" type="revolute">
@@ -54,5 +58,5 @@
     </collision>
     <inertial>
-      <mass value="1"/>
+      <mass value="0.1"/>
       <inertia ixx="0.4" ixy="0.0" ixz="0.0" iyy="0.4" iyz="0.0" izz="0.2"/>
     </inertial>
@@ -81,4 +85,8 @@
       </geometry>
     </collision>
+    <inertial>
+      <mass value="0.1"/>
+      <inertia ixx="0.4" ixy="0.0" ixz="0.0" iyy="0.4" iyz="0.0" izz="0.2"/>
+    </inertial>
   </link>
   <joint name="arm4" type="revolute">
@@ -105,4 +113,8 @@
       </geometry>
     </collision>
+    <inertial>
+      <mass value="0.1"/>
+      <inertia ixx="0.4" ixy="0.0" ixz="0.0" iyy="0.4" iyz="0.0" izz="0.2"/>
+    </inertial>
   </link>
   <joint name="arm3" type="revolute">
@@ -129,4 +141,8 @@
       </geometry>
     </collision>
+    <inertial>
+      <mass value="0.1"/>
+      <inertia ixx="0.4" ixy="0.0" ixz="0.0" iyy="0.4" iyz="0.0" izz="0.2"/>
+    </inertial>
   </link>
   <joint name="arm2" type="revolute">
@@ -153,4 +169,8 @@
       </geometry>
     </collision>
+    <inertial>
+      <mass value="0.1"/>
+      <inertia ixx="0.4" ixy="0.0" ixz="0.0" iyy="0.4" iyz="0.0" izz="0.2"/>
+    </inertial>
   </link>
   <joint name="arm1" type="revolute">
@@ -177,4 +197,8 @@
       </geometry>
     </collision>
+    <inertial>
+      <mass value="0.1"/>
+      <inertia ixx="0.4" ixy="0.0" ixz="0.0" iyy="0.4" iyz="0.0" izz="0.2"/>
+    </inertial>
   </link>
   <joint name="arm1_left" type="continuous">
@@ -201,4 +225,8 @@
       </geometry>
     </collision>
+    <inertial>
+      <mass value="0.1"/>
+      <inertia ixx="0.4" ixy="0.0" ixz="0.0" iyy="0.4" iyz="0.0" izz="0.2"/>
+    </inertial>
   </link>
   <joint name="arm0" type="continuous">
@@ -225,4 +253,8 @@
       </geometry>
     </collision>
+    <inertial>
+      <mass value="0.1"/>
+      <inertia ixx="0.4" ixy="0.0" ixz="0.0" iyy="0.4" iyz="0.0" izz="0.2"/>
+    </inertial>
   </link>
   <joint name="arm0_left" type="continuous">
@@ -249,14 +281,18 @@
       </geometry>
     </collision>
+    <inertial>
+      <mass value="0.1"/>
+      <inertia ixx="0.4" ixy="0.0" ixz="0.0" iyy="0.4" iyz="0.0" izz="0.2"/>
+    </inertial>
   </link>
   <!-- TO-DO: move out to separate file -->
-  <joint name="depth_joint" type="fixed">
+  <!-- <joint name="depth_joint" type="fixed">
     <parent link="link2"/>
     <child link="depth"/>
     <origin rpy="-1.5708 0 -1.5708" xyz="0.044 -0.0115 0.045"/>
   </joint>
-  <link name="depth" />
+  <link name="depth" /> -->
   <!-- TO-DO: move out to separate file -->
-  <ros2_control name="xarm_1s" type="system">
+  <!-- <ros2_control name="xarm_1s" type="system">
     <hardware>
       <plugin>ros2_control_xarm_1s/XArm1SSystemHardware</plugin>
@@ -304,4 +340,4 @@
       <state_interface name="position"/>
     </joint>
-  </ros2_control>
+  </ros2_control> -->
 </robot>
