Commit message: Fixed simulation

File: xarm_moveit_config/config/xarm.ros2_control.xacro (robot description, xacro)
@@ -1,68 +1,69 @@
 <?xml version="1.0"?>
 <robot xmlns:xacro="http://www.ros.org/wiki/xacro">
-    <xacro:macro name="xarm_ros2_control" params="name initial_positions_file simulation_controllers">
-        <xacro:property name="initial_positions" value="${load_yaml(initial_positions_file)['initial_positions']}"/>
-        <!-- <gazebo reference="world">
-        </gazebo>
-        <gazebo>
-        <plugin filename="libgazebo_ros2_control.so" name="gazebo_ros2_control">
-            <parameters>$(arg simulation_controllers)</parameters>
-        </plugin>
-        </gazebo> -->
-        <ros2_control name="${name}" type="system">
-            <hardware>
-                <!-- By default, set up controllers for simulation. This won't work on real hardware -->
-                <plugin>gazebo_ros2_control/GazeboSystem</plugin>
-            </hardware>
-            <joint name="xarm_6_joint">
-                <command_interface name="position"/>
-                <state_interface name="position">
-                  <param name="initial_value">${initial_positions['xarm_6_joint']}</param>
-                </state_interface>
-                <state_interface name="velocity"/>
-            </joint>
-            <joint name="xarm_5_joint">
-                <command_interface name="position"/>
-                <state_interface name="position">
-                  <param name="initial_value">${initial_positions['xarm_5_joint']}</param>
-                </state_interface>
-                <state_interface name="velocity"/>
-            </joint>
-            <joint name="xarm_4_joint">
-                <command_interface name="position"/>
-                <state_interface name="position">
-                  <param name="initial_value">${initial_positions['xarm_4_joint']}</param>
-                </state_interface>
-                <state_interface name="velocity"/>
-            </joint>
-            <joint name="xarm_3_joint">
-                <command_interface name="position"/>
-                <state_interface name="position">
-                  <param name="initial_value">${initial_positions['xarm_3_joint']}</param>
-                </state_interface>
-                <state_interface name="velocity"/>
-            </joint>
-            <joint name="xarm_2_joint">
-                <command_interface name="position"/>
-                <state_interface name="position">
-                  <param name="initial_value">${initial_positions['xarm_2_joint']}</param>
-                </state_interface>
-                <state_interface name="velocity"/>
-            </joint>
-            <joint name="finger_l_joint">
-                <command_interface name="position"/>
-                <state_interface name="position">
-                  <param name="initial_value">${initial_positions['finger_l_joint']}</param>
-                </state_interface>
-                <state_interface name="velocity"/>
-            </joint>
-            <joint name="finger_r_joint">
-                <command_interface name="position"/>
-                <state_interface name="position">
-                  <param name="initial_value">${initial_positions['finger_r_joint']}</param>
-                </state_interface>
-                <state_interface name="velocity"/>
-            </joint>
-        </ros2_control>
-    </xacro:macro>
+  <xacro:macro name="xarm_ros2_control" params="name initial_positions_file simulation_controllers">
+    <xacro:property name="initial_positions"
+      value="${xacro.load_yaml(initial_positions_file)['initial_positions']}" />
+    <gazebo reference="world">
+    </gazebo>
+    <gazebo>
+      <plugin filename="libgazebo_ros2_control.so" name="gazebo_ros2_control">
+        <parameters>$(arg simulation_controllers)</parameters>
+      </plugin>
+    </gazebo>
+    <ros2_control name="${name}" type="system">
+      <hardware>
+        <!-- By default, set up controllers for simulation. This won't work on real hardware -->
+        <plugin>gazebo_ros2_control/GazeboSystem</plugin>
+      </hardware>
+      <joint name="xarm_6_joint">
+        <command_interface name="position" />
+        <state_interface name="position">
+          <param name="initial_value">${initial_positions['xarm_6_joint']}</param>
+        </state_interface>
+        <state_interface name="velocity" />
+      </joint>
+      <joint name="xarm_5_joint">
+        <command_interface name="position" />
+        <state_interface name="position">
+          <param name="initial_value">${initial_positions['xarm_5_joint']}</param>
+        </state_interface>
+        <state_interface name="velocity" />
+      </joint>
+      <joint name="xarm_4_joint">
+        <command_interface name="position" />
+        <state_interface name="position">
+          <param name="initial_value">${initial_positions['xarm_4_joint']}</param>
+        </state_interface>
+        <state_interface name="velocity" />
+      </joint>
+      <joint name="xarm_3_joint">
+        <command_interface name="position" />
+        <state_interface name="position">
+          <param name="initial_value">${initial_positions['xarm_3_joint']}</param>
+        </state_interface>
+        <state_interface name="velocity" />
+      </joint>
+      <joint name="xarm_2_joint">
+        <command_interface name="position" />
+        <state_interface name="position">
+          <param name="initial_value">${initial_positions['xarm_2_joint']}</param>
+        </state_interface>
+        <state_interface name="velocity" />
+      </joint>
+      <joint name="finger_l_joint">
+        <command_interface name="position" />
+        <state_interface name="position">
+          <param name="initial_value">${initial_positions['finger_l_joint']}</param>
+        </state_interface>
+        <state_interface name="velocity" />
+      </joint>
+      <joint name="finger_r_joint">
+        <command_interface name="position" />
+        <state_interface name="position">
+          <param name="initial_value">${initial_positions['finger_r_joint']}</param>
+        </state_interface>
+        <state_interface name="velocity" />
+      </joint>
+    </ros2_control>
+  </xacro:macro>
 </robot>

File: xarm_moveit_config/config/xarm.urdf.xacro (robot description, xacro)
@@ -2,12 +2,13 @@
 <robot xmlns:xacro="http://www.ros.org/wiki/xacro" name="xarm">
     <xacro:arg name="initial_positions_file" default="initial_positions.yaml" />
+    <xacro:arg name="simulation_controllers" default="" />
     <!-- Import xarm urdf file -->
     <xacro:include filename="$(find xarm_description)/urdf/xarm_world.urdf.xacro" />
     <!-- Import control_xacro -->
     <xacro:include filename="xarm.ros2_control.xacro" />
+    <!-- <xacro:xarm_ros2_control name="GazeboSystem"
+        initial_positions_file="$(arg initial_positions_file)" /> -->
     <xacro:xarm_ros2_control name="GazeboSystem"
-        initial_positions_file="$(arg initial_positions_file)" />
-    <!-- <xacro:ur_ros2_control name="GazeboSystem"
         initial_positions_file="$(arg initial_positions_file)"
-        simulation_controllers="$(arg simulation_controllers)" /> -->
+        simulation_controllers="$(arg simulation_controllers)" />
 </robot>

Commit message: Added support package for real robot setup

File: xarm_moveit_config/config/xarm.ros2_control.xacro (robot description, xacro)
@@ -1,69 +1,132 @@
 <?xml version="1.0"?>
 <robot xmlns:xacro="http://www.ros.org/wiki/xacro">
-  <xacro:macro name="xarm_ros2_control" params="name initial_positions_file simulation_controllers">
+  <xacro:macro name="xarm_ros2_control" params="name initial_positions_file controllers sim_robot">
     <xacro:property name="initial_positions"
       value="${xacro.load_yaml(initial_positions_file)['initial_positions']}" />
-    <gazebo reference="world">
-    </gazebo>
-    <gazebo>
-      <plugin filename="libgazebo_ros2_control.so" name="gazebo_ros2_control">
-        <parameters>$(arg simulation_controllers)</parameters>
-      </plugin>
-    </gazebo>
-    <ros2_control name="${name}" type="system">
-      <hardware>
-        <!-- By default, set up controllers for simulation. This won't work on real hardware -->
-        <plugin>gazebo_ros2_control/GazeboSystem</plugin>
-      </hardware>
-      <joint name="xarm_6_joint">
-        <command_interface name="position" />
-        <state_interface name="position">
-          <param name="initial_value">${initial_positions['xarm_6_joint']}</param>
-        </state_interface>
-        <state_interface name="velocity" />
-      </joint>
-      <joint name="xarm_5_joint">
-        <command_interface name="position" />
-        <state_interface name="position">
-          <param name="initial_value">${initial_positions['xarm_5_joint']}</param>
-        </state_interface>
-        <state_interface name="velocity" />
-      </joint>
-      <joint name="xarm_4_joint">
-        <command_interface name="position" />
-        <state_interface name="position">
-          <param name="initial_value">${initial_positions['xarm_4_joint']}</param>
-        </state_interface>
-        <state_interface name="velocity" />
-      </joint>
-      <joint name="xarm_3_joint">
-        <command_interface name="position" />
-        <state_interface name="position">
-          <param name="initial_value">${initial_positions['xarm_3_joint']}</param>
-        </state_interface>
-        <state_interface name="velocity" />
-      </joint>
-      <joint name="xarm_2_joint">
-        <command_interface name="position" />
-        <state_interface name="position">
-          <param name="initial_value">${initial_positions['xarm_2_joint']}</param>
-        </state_interface>
-        <state_interface name="velocity" />
-      </joint>
-      <joint name="finger_l_joint">
-        <command_interface name="position" />
-        <state_interface name="position">
-          <param name="initial_value">${initial_positions['finger_l_joint']}</param>
-        </state_interface>
-        <state_interface name="velocity" />
-      </joint>
-      <joint name="finger_r_joint">
-        <command_interface name="position" />
-        <state_interface name="position">
-          <param name="initial_value">${initial_positions['finger_r_joint']}</param>
-        </state_interface>
-        <state_interface name="velocity" />
-      </joint>
-    </ros2_control>
+    <xacro:if value="${sim_robot}">
+      <gazebo reference="world">
+      </gazebo>
+      <gazebo>
+        <plugin filename="libgazebo_ros2_control.so" name="gazebo_ros2_control">
+          <parameters>$(arg controllers)</parameters>
+        </plugin>
+      </gazebo>
+      <ros2_control name="GazeboSystem" type="system">
+        <hardware>
+          <!-- By default, set up controllers for simulation. This won't work on real hardware -->
+          <plugin>gazebo_ros2_control/GazeboSystem</plugin>
+        </hardware>
+        <joint name="xarm_6_joint">
+          <command_interface name="position" />
+          <state_interface name="position">
+            <param name="initial_value">${initial_positions['xarm_6_joint']}</param>
+          </state_interface>
+          <state_interface name="velocity" />
+        </joint>
+        <joint name="xarm_5_joint">
+          <command_interface name="position" />
+          <state_interface name="position">
+            <param name="initial_value">${initial_positions['xarm_5_joint']}</param>
+          </state_interface>
+          <state_interface name="velocity" />
+        </joint>
+        <joint name="xarm_4_joint">
+          <command_interface name="position" />
+          <state_interface name="position">
+            <param name="initial_value">${initial_positions['xarm_4_joint']}</param>
+          </state_interface>
+          <state_interface name="velocity" />
+        </joint>
+        <joint name="xarm_3_joint">
+          <command_interface name="position" />
+          <state_interface name="position">
+            <param name="initial_value">${initial_positions['xarm_3_joint']}</param>
+          </state_interface>
+          <state_interface name="velocity" />
+        </joint>
+        <joint name="xarm_2_joint">
+          <command_interface name="position" />
+          <state_interface name="position">
+            <param name="initial_value">${initial_positions['xarm_2_joint']}</param>
+          </state_interface>
+          <state_interface name="velocity" />
+        </joint>
+        <joint name="finger_l_joint">
+          <command_interface name="position" />
+          <state_interface name="position">
+            <param name="initial_value">${initial_positions['finger_l_joint']}</param>
+          </state_interface>
+          <state_interface name="velocity" />
+        </joint>
+        <joint name="finger_r_joint">
+          <command_interface name="position" />
+          <state_interface name="position">
+            <param name="initial_value">${initial_positions['finger_r_joint']}</param>
+          </state_interface>
+          <state_interface name="velocity" />
+        </joint>
+      </ros2_control>
+    </xacro:if>
+    <xacro:unless value="${sim_robot}">
+      <ros2_control name="${name}" type="system">
+        <hardware>
+          <plugin>topic_based_ros2_control/TopicBasedSystem</plugin>
+          <param name="joint_commands_topic">/multi_servo_cmd_sub</param>
+          <param name="joint_states_topic">/servo_pos_publisher</param>
+          <param name="sum_wrapped_joint_states">true</param>
+        </hardware>
+        <joint name="xarm_6_joint">
+          <command_interface name="position" />
+          <state_interface name="position">
+            <param name="initial_value">${initial_positions['xarm_6_joint']}</param>
+          </state_interface>
+          <state_interface name="velocity" />
+        </joint>
+        <joint name="xarm_5_joint">
+          <command_interface name="position" />
+          <state_interface name="position">
+            <param name="initial_value">${initial_positions['xarm_5_joint']}</param>
+          </state_interface>
+          <state_interface name="velocity" />
+        </joint>
+        <joint name="xarm_4_joint">
+          <command_interface name="position" />
+          <state_interface name="position">
+            <param name="initial_value">${initial_positions['xarm_4_joint']}</param>
+          </state_interface>
+          <state_interface name="velocity" />
+        </joint>
+        <joint name="xarm_3_joint">
+          <command_interface name="position" />
+          <state_interface name="position">
+            <param name="initial_value">${initial_positions['xarm_3_joint']}</param>
+          </state_interface>
+          <state_interface name="velocity" />
+        </joint>
+        <joint name="xarm_2_joint">
+          <command_interface name="position" />
+          <state_interface name="position">
+            <param name="initial_value">${initial_positions['xarm_2_joint']}</param>
+          </state_interface>
+          <state_interface name="velocity" />
+        </joint>
+        <joint name="finger_l_joint">
+          <command_interface name="position" />
+          <state_interface name="position">
+            <param name="initial_value">${initial_positions['finger_l_joint']}</param>
+          </state_interface>
+          <state_interface name="velocity" />
+        </joint>
+        <joint name="finger_r_joint">
+          <param name="mimic">finger_l_joint</param>
+          <param name="multiplier">1</param>
+          <command_interface name="position" />
+          <state_interface name="position">
+            <param name="initial_value">${initial_positions['finger_r_joint']}</param>
+          </state_interface>
+          <state_interface name="velocity" />
+        </joint>
+      </ros2_control>
+    </xacro:unless>
   </xacro:macro>
 </robot>

File: xarm_moveit_config/config/xarm.urdf.xacro (robot description, xacro)
@@ -2,13 +2,13 @@
 <robot xmlns:xacro="http://www.ros.org/wiki/xacro" name="xarm">
     <xacro:arg name="initial_positions_file" default="initial_positions.yaml" />
-    <xacro:arg name="simulation_controllers" default="" />
+    <xacro:arg name="controllers" default="" />
+    <xacro:arg name="sim_robot" default="false"/>
     <!-- Import xarm urdf file -->
     <xacro:include filename="$(find xarm_description)/urdf/xarm_world.urdf.xacro" />
     <!-- Import control_xacro -->
     <xacro:include filename="xarm.ros2_control.xacro" />
-    <!-- <xacro:xarm_ros2_control name="GazeboSystem"
-        initial_positions_file="$(arg initial_positions_file)" /> -->
-    <xacro:xarm_ros2_control name="GazeboSystem"
+    <xacro:xarm_ros2_control name="System"
         initial_positions_file="$(arg initial_positions_file)"
-        simulation_controllers="$(arg simulation_controllers)" />
+        controllers="$(arg controllers)"
+        sim_robot="$(arg sim_robot)"/>
 </robot>
