Commit message: Feat: Added ros2_control and serial communication for real robot

File: xarm_moveit_config/config/xarm.ros2_control.xacro (robot description, xacro)
@@ -1,98 +1,107 @@
 <?xml version="1.0"?>
 <robot xmlns:xacro="http://www.ros.org/wiki/xacro">
-    <xacro:macro name="xarm_ros2_control" params="name initial_positions_file is_simulation">
-        <xacro:property name="initial_positions" value="${xacro.load_yaml(initial_positions_file)['initial_positions']}"/>
-        <gazebo>
-          <plugin filename="libgz_ros2_control-system.so" name="gz_ros2_control::GazeboSimROS2ControlPlugin">
-            <parameters>$(find xarm_moveit_config)/config/ros2_controllers.yaml</parameters>
-          </plugin>
-        </gazebo>
-        <ros2_control name="${name}" type="system">
-            <hardware>
-                <!-- By default, set up controllers for simulation. This won't work on real hardware -->
-                <xacro:if value="${is_simulation}">
-                  <plugin>gz_ros2_control/GazeboSimSystem</plugin>
-                </xacro:if>
-                <xacro:unless value="${is_simulation}">
-                  <plugin>mock_components/GenericSystem</plugin>
-                </xacro:unless>
-            </hardware>
-            <joint name="arm6">
-                <command_interface name="position">
-                  <param name="min">-2.09439435</param>
-                  <param name="max">2.09439435</param>
-                </command_interface>
-                <state_interface name="position">
-                  <param name="initial_value">${initial_positions['arm6']}</param>
-                </state_interface>
-                <state_interface name="velocity"/>
-            </joint>
-            <joint name="arm5">
-                <command_interface name="position">
-                  <param name="min">-2.09439435</param>
-                  <param name="max">2.09439435</param>
-                </command_interface>
-                <state_interface name="position">
-                  <param name="initial_value">${initial_positions['arm5']}</param>
-                </state_interface>
-                <state_interface name="velocity"/>
-            </joint>
-            <joint name="arm4">
-                <command_interface name="position">
-                  <param name="min">-2.09439435</param>
-                  <param name="max">2.09439435</param>
-                </command_interface>
-                <state_interface name="position">
-                  <param name="initial_value">${initial_positions['arm4']}</param>
-                </state_interface>
-                <state_interface name="velocity"/>
-            </joint>
-            <joint name="arm3">
-                <command_interface name="position">
-                  <param name="min">-2.09439435</param>
-                  <param name="max">2.09439435</param>
-                </command_interface>
-                <state_interface name="position">
-                  <param name="initial_value">${initial_positions['arm3']}</param>
-                </state_interface>
-                <state_interface name="velocity"/>
-            </joint>
-            <joint name="arm2">
-                <command_interface name="position">
-                  <param name="min">-2.09439435</param>
-                  <param name="max">2.09439435</param>
-                </command_interface>
-                <state_interface name="position">
-                  <param name="initial_value">${initial_positions['arm2']}</param>
-                </state_interface>
-                <state_interface name="velocity"/>
-            </joint>
-            <joint name="arm1">
-                <command_interface name="position">
-                  <param name="min">0</param>
-                  <param name="max">0.8464847</param>
-                </command_interface>
-                <state_interface name="position">
-                  <param name="initial_value">${initial_positions['arm1']}</param>
-                </state_interface>
-                <state_interface name="velocity"/>
-            </joint>
-            <joint name="arm1_left">
-                <state_interface name="position"/>
-                <state_interface name="velocity"/>
-            </joint>
-            <joint name="arm0">
-                <state_interface name="position">
-                  <param name="initial_value">-0.3</param>
-                </state_interface>
-                <state_interface name="velocity"/>
-            </joint>
-            <joint name="arm0_left">
-                <state_interface name="position">
-                  <param name="initial_value">0.3</param>
-                </state_interface>
-                <state_interface name="velocity"/>
-            </joint>
-        </ros2_control>
-    </xacro:macro>
+  <xacro:macro name="xarm_ros2_control" params="name initial_positions_file is_simulation">
+    <xacro:property name="initial_positions"
+      value="${xacro.load_yaml(initial_positions_file)['initial_positions']}" />
+    <xacro:if value="${is_simulation}">
+      <gazebo>
+        <plugin filename="libgz_ros2_control-system.so"
+          name="gz_ros2_control::GazeboSimROS2ControlPlugin">
+          <parameters>$(find xarm_moveit_config)/config/ros2_controllers.yaml</parameters>
+        </plugin>
+      </gazebo>
+    </xacro:if>
+    <ros2_control name="${name}" type="system">
+      <hardware>
+        <!-- By default, set up controllers for simulation. This won't work on real hardware -->
+        <xacro:if value="${is_simulation}">
+          <plugin>gz_ros2_control/GazeboSimSystem</plugin>
+        </xacro:if>
+        <xacro:unless value="${is_simulation}">
+          <plugin>xarm_control/XArmSystemHardware</plugin>
+          <param name="device">/dev/ttyUSB0</param>
+          <param name="zero_pos">11750 12250 11750 12000 11000 16800</param>
+          <param name="baud_rate">230400</param>
+          <param name="timeout_ms">1000</param>
+          <param name="reduction">15.0</param>
+        </xacro:unless>
+      </hardware>
+      <joint name="arm6">
+        <command_interface name="position">
+          <param name="min">-1.92</param>
+          <param name="max">1.92</param>
+        </command_interface>
+        <state_interface name="position">
+          <param name="initial_value">${initial_positions['arm6']}</param>
+        </state_interface>
+        <state_interface name="velocity" />
+      </joint>
+      <joint name="arm5">
+        <command_interface name="position">
+          <param name="min">-1.92</param>
+          <param name="max">1.92</param>
+        </command_interface>
+        <state_interface name="position">
+          <param name="initial_value">${initial_positions['arm5']}</param>
+        </state_interface>
+        <state_interface name="velocity" />
+      </joint>
+      <joint name="arm4">
+        <command_interface name="position">
+          <param name="min">-1.92</param>
+          <param name="max">1.92</param>
+        </command_interface>
+        <state_interface name="position">
+          <param name="initial_value">${initial_positions['arm4']}</param>
+        </state_interface>
+        <state_interface name="velocity" />
+      </joint>
+      <joint name="arm3">
+        <command_interface name="position">
+          <param name="min">-1.92</param>
+          <param name="max">1.92</param>
+        </command_interface>
+        <state_interface name="position">
+          <param name="initial_value">${initial_positions['arm3']}</param>
+        </state_interface>
+        <state_interface name="velocity" />
+      </joint>
+      <joint name="arm2">
+        <command_interface name="position">
+          <param name="min">-1.92</param>
+          <param name="max">1.92</param>
+        </command_interface>
+        <state_interface name="position">
+          <param name="initial_value">${initial_positions['arm2']}</param>
+        </state_interface>
+        <state_interface name="velocity" />
+      </joint>
+      <joint name="arm1">
+        <command_interface name="position">
+          <param name="min">0</param>
+          <param name="max">0.8464847</param>
+        </command_interface>
+        <state_interface name="position">
+          <param name="initial_value">${initial_positions['arm1']}</param>
+        </state_interface>
+        <state_interface name="velocity" />
+      </joint>
+      <!-- <joint name="arm1_left">
+        <state_interface name="position" />
+        <state_interface name="velocity" />
+      </joint>
+      <joint name="arm0">
+        <state_interface name="position">
+          <param name="initial_value">-0.3</param>
+        </state_interface>
+        <state_interface name="velocity" />
+      </joint>
+      <joint name="arm0_left">
+        <state_interface name="position">
+          <param name="initial_value">0.3</param>
+        </state_interface>
+        <state_interface name="velocity" />
+      </joint> -->
+    </ros2_control>
+  </xacro:macro>
 </robot>

File: xarm_moveit_config/config/xarm.urdf.xacro (robot description, xacro)
@@ -11,5 +11,5 @@
     </xacro:if>
     <xacro:unless value="$(arg is_simulation)">
-        <xacro:xarm_ros2_control name="FakeSystem" initial_positions_file="$(arg initial_positions_file)" is_simulation="$(arg is_simulation)"/>
+        <xacro:xarm_ros2_control name="xarm_control" initial_positions_file="$(arg initial_positions_file)" is_simulation="$(arg is_simulation)"/>
     </xacro:unless>
 </robot>

Commit message: Fix: Modified ros2_control xacro file to work with both simulated and real robot

File: xarm_moveit_config/config/xarm.ros2_control.xacro (robot description, xacro)
@@ -87,20 +87,22 @@
         <state_interface name="velocity" />
       </joint>
-      <!-- <joint name="arm1_left">
-        <state_interface name="position" />
-        <state_interface name="velocity" />
-      </joint>
-      <joint name="arm0">
-        <state_interface name="position">
-          <param name="initial_value">-0.3</param>
-        </state_interface>
-        <state_interface name="velocity" />
-      </joint>
-      <joint name="arm0_left">
-        <state_interface name="position">
-          <param name="initial_value">0.3</param>
-        </state_interface>
-        <state_interface name="velocity" />
-      </joint> -->
+      <xacro:if value="${is_simulation}">
+        <joint name="arm1_left">
+          <state_interface name="position" />
+          <state_interface name="velocity" />
+        </joint>
+        <joint name="arm0">
+          <state_interface name="position">
+            <param name="initial_value">-0.3</param>
+          </state_interface>
+          <state_interface name="velocity" />
+        </joint>
+        <joint name="arm0_left">
+          <state_interface name="position">
+            <param name="initial_value">0.3</param>
+          </state_interface>
+          <state_interface name="velocity" />
+        </joint>
+      </xacro:if>
     </ros2_control>
   </xacro:macro>
