Commit message: Remove unnecessary files

File: xarm_description/urdf/xarm.urdf.xacro (robot description, xacro)
@@ -1,196 +1,343 @@
 <?xml version="1.0" ?>
 <robot xmlns:xacro="http://www.ros.org/wiki/xacro" name="xarm">
-    <xacro:include filename="$(find xarm_description)/urdf/gripper.urdf.xacro"/>
-    <material name="DarkGrey">
-        <color rgba="0.3 0.3 0.3 1.0" />
-    </material>
-    <material name="Red">
-        <color rgba="0.3 0.3 0.3 1.0" />
-    </material>
-    <material name="Black">
-        <color rgba="0 0 0 1.0" />
-    </material>
-    <material name="Orange">
-        <color rgba="0.0 0.15 0.7 1.0" />
-    </material>
-    <material name="Silver">
-        <color rgba="1.0 1.0 1.0 1.0" />
-    </material>
-    <material name="Grey">
-        <color rgba="0.7 0.7 0.7 1.0" />
-    </material>
-    <material name="Blue">
-        <color rgba="0.0 0.0 0.8 1.0" />
-    </material>
-    <material name="HandGray">
-        <color rgba="0.953 0.996 0.694 1.0" />
-    </material>
-    <material name="SickBlue">
-        <color rgba="0.3058 0.5921 0.7294 1.0" />
-    </material>
-    <property name="M_PI" value="3.1415926535897931" />
-    <link name="xarm_base_link">
-        <visual>
-            <origin rpy="0 0 0" xyz="0.0 0.0 0.0" />
-            <geometry>
-                <mesh filename="file://$(find xarm_description)/meshes/stls/base.stl" scale="1.0 1.0 1.0" />
-            </geometry>
-            <material name="Blue" />
-        </visual>
-        <collision>
-            <origin rpy="0 0 0" xyz="0 0 0" />
-            <geometry>
-                <mesh filename="file://$(find xarm_description)/meshes/stls/base.stl" scale="1.0 1.0 1.0" />
-            </geometry>
-        </collision>
-        <inertial>
-            <mass value="0.1" />
-            <inertia ixx="0.03" iyy="0.03" izz="0.03" ixy="0.0" ixz="0.0" iyz="0.0" />
-        </inertial>
-    </link>
-    <link name="xarm_6_link">
-        <visual>
-            <origin rpy="0 0 0" xyz="0.0 0.0 0.0" />
-            <geometry>
-                <mesh filename="file://$(find xarm_description)/meshes/stls/link6.stl" scale="1.0 1.0 1.0" />
-            </geometry>
-            <material name="DarkGrey" />
-        </visual>
-        <collision>
-            <origin rpy="0 0 0" xyz="0.0 0.0 0.0" />
-            <geometry>
-                <mesh filename="file://$(find xarm_description)/meshes/stls/link6.stl" scale="1.0 1.0 1.0" />
-            </geometry>
-        </collision>
-        <inertial>
-            <mass value="0.1" />
-            <inertia ixx="0.03" iyy="0.03" izz="0.03" ixy="0.0" ixz="0.0" iyz="0.0" />
-        </inertial>
-    </link>
-    <link name="xarm_5_link">
-        <visual>
-            <origin rpy="0 0 0" xyz="0.0 0.0 0.0" />
-            <geometry>
-                <mesh filename="file://$(find xarm_description)/meshes/stls/link5.stl" scale="1.0 1.0 1.0" />
-            </geometry>
-            <material name="Blue" />
-        </visual>
-        <collision>
-            <origin rpy="0 0 0" xyz="0.0 0.0 0.0" />
-            <geometry>
-                <mesh filename="file://$(find xarm_description)/meshes/stls/link5.stl" scale="1.0 1.0 1.0" />
-            </geometry>
-        </collision>
-        <inertial>
-            <mass value="0.1" />
-            <inertia ixx="0.03" iyy="0.03" izz="0.03" ixy="0.0" ixz="0.0" iyz="0.0" />
-        </inertial>
-    </link>
-    <link name="xarm_4_link">
-        <visual>
-            <origin rpy="0 0 0" xyz="0.0 0.0 0.0" />
-            <geometry>
-                <mesh filename="file://$(find xarm_description)/meshes/stls/link4.stl" scale="1.0 1.0 1.0" />
-            </geometry>
-            <material name="DarkGrey" />
-        </visual>
-        <collision>
-            <origin rpy="0 0 0" xyz="0.0 0.0 0.0" />
-            <geometry>
-                <mesh filename="file://$(find xarm_description)/meshes/stls/link4.stl" scale="1.0 1.0 1.0" />
-            </geometry>
-        </collision>
-        <inertial>
-            <mass value="0.1" />
-            <inertia ixx="0.03" iyy="0.03" izz="0.03" ixy="0.0" ixz="0.0" iyz="0.0" />
-        </inertial>
-    </link>
-    <link name="xarm_3_link">
-        <visual>
-            <origin rpy="0 0 0" xyz="0.0 0.0 0.0" />
-            <geometry>
-                <mesh filename="file://$(find xarm_description)/meshes/stls/link3.stl" scale="1.0 1.0 1.0" />
-            </geometry>
-            <material name="Blue" />
-        </visual>
-        <collision>
-            <origin rpy="0 0 0" xyz="0.0 0.0 0.0" />
-            <geometry>
-                <mesh filename="file://$(find xarm_description)/meshes/stls/link3.stl" scale="1.0 1.0 1.0" />
-            </geometry>
-        </collision>
-        <inertial>
-            <mass value="0.1" />
-            <inertia ixx="0.03" iyy="0.03" izz="0.03" ixy="0.0" ixz="0.0" iyz="0.0" />
-        </inertial>
-    </link>
-    <link name="xarm_2_link">
-        <visual>
-            <origin rpy="0 0 0" xyz="0.0 0.0 0.0" />
-            <geometry>
-                <mesh filename="file://$(find xarm_description)/meshes/stls/link2.stl" scale="1.0 1.0 1.0" />
-            </geometry>
-            <material name="DarkGrey" />
-        </visual>
-        <collision>
-            <origin rpy="0 0 0" xyz="0.0 0.0 0.0" />
-            <geometry>
-                <mesh filename="file://$(find xarm_description)/meshes/stls/link2.stl" scale="1.0 1.0 1.0" />
-            </geometry>
-        </collision>
-        <inertial>
-            <mass value="0.1" />
-            <inertia ixx="0.03" iyy="0.03" izz="0.03" ixy="0.0" ixz="0.0" iyz="0.0" />
-        </inertial>
-    </link>
-    <joint name="xarm_6_joint" type="revolute">
-        <origin rpy="0 0 0" xyz="0 0.0 0.03603" />
-        <axis xyz="0 0 1" />
-        <limit effort="1000" lower="-1.737238322" upper="1.79965407" velocity="1.0" />
-        <!--safety_controller k_position="30" k_velocity="30" soft_lower_limit="-2.93215314335" soft_upper_limit="2.93215314335"/>
-        <dynamics damping="1.0"/-->
-        <parent link="xarm_base_link" />
-        <child link="xarm_6_link" />
-    </joint>
-    <joint name="xarm_5_joint" type="revolute">
-        <origin rpy="0 0 0" xyz="0 -0.0022 0.03195" />
-        <axis xyz="1 0 0" />
-        <limit effort="1000" lower="-1.592023304" upper="1.86797401" velocity="1.0" />
-        <!--safety_controller k_position="30" k_velocity="30" soft_lower_limit="-2.93215314335" soft_upper_limit="2.93215314335"/>
-        <dynamics damping="1.0"/-->
-        <parent link="xarm_6_link" />
-        <child link="xarm_5_link" />
-    </joint>
-    <joint name="xarm_4_joint" type="revolute">
-        <origin rpy="0 0 0" xyz="0 0.0 0.09765" />
-        <axis xyz="1 0 0" />
-        <limit effort="1000" lower="-1.910427965" upper="1.910427965" velocity="1.0" />
-        <!--safety_controller k_position="30" k_velocity="30" soft_lower_limit="-2.93215314335" soft_upper_limit="2.93215314335"/>
-        <dynamics damping="1.0"/-->
-        <parent link="xarm_5_link" />
-        <child link="xarm_4_link" />
-    </joint>
-    <joint name="xarm_3_joint" type="revolute">
-        <origin rpy="0 0 0" xyz="0 0.0 0.09825" />
-        <axis xyz="1 0 0" />
-        <limit effort="1000" lower="-1.740612146" upper="1.86797401" velocity="1.0" />
-        <!--safety_controller k_position="30" k_velocity="30" soft_lower_limit="-2.93215314335" soft_upper_limit="2.93215314335"/>
-        <dynamics damping="1.0"/-->
-        <parent link="xarm_4_link" />
-        <child link="xarm_3_link" />
-    </joint>
-    <joint name="xarm_2_joint" type="revolute">
-        <origin rpy="0 0 0" xyz="0 -0.001205 0.05306" />
-        <axis xyz="0 0 1" />
-        <limit effort="1000" lower="-2.17494876" upper="1.63121157" velocity="1.0" />
-        <!--safety_controller k_position="30" k_velocity="30" soft_lower_limit="-2.93215314335" soft_upper_limit="2.93215314335"/>
-        <dynamics damping="1.0"/-->
-        <parent link="xarm_3_link" />
-        <child link="xarm_2_link" />
-    </joint>
-    <joint name="gripper_joint" type="fixed">
-        <origin xyz="0.0 0.0 0.006" rpy="0.0 -1.57 1.57"/>
-        <parent link="xarm_2_link"/>
-        <child link="gripper_base"/>
-    </joint>
+  <material name="black">
+    <color rgba="0.2 0.2 0.2 1"/>
+  </material>
+  <material name="blue">
+    <color rgba="0.3 0.5 0.9 1.0"/>
+  </material>
+  <link name="world"/>
+  <joint name="world_joint" type="fixed">
+    <parent link="world"/>
+    <child link="base_link"/>
+    <origin rpy="0.0 0.0 0.0" xyz="0.0 0.0 0.0"/>
+  </joint>
+  <link name="base_link">
+    <visual>
+      <origin rpy="0 0 0" xyz="0.0 0.0 0.0" />
+      <geometry>
+        <!-- <mesh filename="package://xarm_description/meshes/base.stl" scale="1.0 1.0 1.0" /> -->
+        <mesh filename="file://$(find xarm_description)/meshes/base.stl" scale="1.0 1.0 1.0" />
+      </geometry>
+      <material name="blue" />
+    </visual>
+    <collision>
+      <origin rpy="0 0 0" xyz="0 0 0" />
+      <geometry>
+        <!-- <mesh filename="package://xarm_description/meshes/base_collision.stl" scale="1.0 1.0 1.0" /> -->
+        <mesh filename="file://$(find xarm_description)/meshes/base_collision.stl" scale="1.0 1.0 1.0" />
+      </geometry>
+    </collision>
+    <inertial>
+      <mass value="0.1"/>
+      <inertia ixx="0.4" ixy="0.0" ixz="0.0" iyy="0.4" iyz="0.0" izz="0.2"/>
+    </inertial>
+  </link>
+  <joint name="arm6" type="revolute">
+    <limit effort="1000" lower="-2.1" upper="2.1" velocity="1.0" />
+    <parent link="base_link"/>
+    <child link="link6"/>
+    <origin rpy="0.0 0.0 0.0" xyz="0.0 0.0 0.043"/>
+    <axis xyz="0 0 1"/>
+  </joint>
+  <link name="link6">
+    <visual>
+      <origin rpy="0 0 0" xyz="0.0 0.0 0.0" />
+      <geometry>
+        <!-- <mesh filename="package://xarm_description/meshes/link6.stl" scale="1.0 1.0 1.0" /> -->
+        <mesh filename="file://$(find xarm_description)/meshes/link6.stl" scale="1.0 1.0 1.0" />
+      </geometry>
+      <material name="blue" />
+    </visual>
+    <collision>
+      <origin rpy="0 0 0" xyz="0 0 0" />
+      <geometry>
+        <!-- <mesh filename="package://xarm_description/meshes/link6_collision.stl" scale="1.0 1.0 1.0" /> -->
+        <mesh filename="file://$(find xarm_description)/meshes/link6_collision.stl" scale="1.0 1.0 1.0" />
+      </geometry>
+    </collision>
+    <inertial>
+      <mass value="0.1"/>
+      <inertia ixx="0.4" ixy="0.0" ixz="0.0" iyy="0.4" iyz="0.0" izz="0.2"/>
+    </inertial>
+  </link>
+  <joint name="arm5" type="revolute">
+    <limit effort="1000" lower="-1.5708" upper="1.5708" velocity="1.0" />
+    <parent link="link6"/>
+    <child link="link5"/>
+    <origin rpy="0.0 0.0 0.0" xyz="0.002 0.0 0.032"/>
+    <axis xyz="0 1 0"/>
+  </joint>
+  <link name="link5">
+    <visual>
+      <origin rpy="0 0 0" xyz="0.0 0.0 0.0" />
+      <geometry>
+        <!-- <mesh filename="package://xarm_description/meshes/link5.stl" scale="1.0 1.0 1.0" /> -->
+        <mesh filename="file://$(find xarm_description)/meshes/link5.stl" scale="1.0 1.0 1.0" />
+      </geometry>
+      <material name="blue" />
+    </visual>
+    <collision>
+      <origin rpy="0 0 0" xyz="0 0 0" />
+      <geometry>
+        <!-- <mesh filename="package://xarm_description/meshes/link5_collision.stl" scale="1.0 1.0 1.0" /> -->
+        <mesh filename="file://$(find xarm_description)/meshes/link5_collision.stl" scale="1.0 1.0 1.0" />
+      </geometry>
+    </collision>
+    <inertial>
+      <mass value="0.1"/>
+      <inertia ixx="0.4" ixy="0.0" ixz="0.0" iyy="0.4" iyz="0.0" izz="0.2"/>
+    </inertial>
+  </link>
+  <joint name="arm4" type="revolute">
+    <limit effort="1000" lower="-2.09" upper="2.09" velocity="1.0" />
+    <parent link="link5"/>
+    <child link="link4"/>
+    <origin rpy="0.0 0.0 0.0" xyz="0.0 0.0 0.09775"/>
+    <axis xyz="0 1 0"/>
+  </joint>
+  <link name="link4">
+    <visual>
+      <origin rpy="0 0 0" xyz="0.0 0.0 0.0" />
+      <geometry>
+        <!-- <mesh filename="package://xarm_description/meshes/link4.stl" scale="1.0 1.0 1.0" /> -->
+        <mesh filename="file://$(find xarm_description)/meshes/link4.stl" scale="1.0 1.0 1.0" />
+      </geometry>
+      <material name="black" />
+    </visual>
+    <collision>
+      <origin rpy="0 0 0" xyz="0 0 0" />
+      <geometry>
+        <!-- <mesh filename="package://xarm_description/meshes/link4_collision.stl" scale="1.0 1.0 1.0" /> -->
+        <mesh filename="file://$(find xarm_description)/meshes/link4_collision.stl" scale="1.0 1.0 1.0" />
+      </geometry>
+    </collision>
+    <inertial>
+      <mass value="0.1"/>
+      <inertia ixx="0.4" ixy="0.0" ixz="0.0" iyy="0.4" iyz="0.0" izz="0.2"/>
+    </inertial>
+  </link>
+  <joint name="arm3" type="revolute">
+    <limit effort="1000" lower="-1.85" upper="2.07" velocity="1.0" />
+    <parent link="link4"/>
+    <child link="link3"/>
+    <origin rpy="0.0 0.0 0.0" xyz="0.0 0.0 0.099"/>
+    <axis xyz="0 1 0"/>
+  </joint>
+  <link name="link3">
+    <visual>
+      <origin rpy="0 0 0" xyz="0.0 0.0 0.0" />
+      <geometry>
+        <!-- <mesh filename="package://xarm_description/meshes/link3.stl" scale="1.0 1.0 1.0" /> -->
+        <mesh filename="file://$(find xarm_description)/meshes/link3.stl" scale="1.0 1.0 1.0" />
+      </geometry>
+      <material name="blue" />
+    </visual>
+    <collision>
+      <origin rpy="0 0 0" xyz="0 0 0" />
+      <geometry>
+        <!-- <mesh filename="package://xarm_description/meshes/link3_collision.stl" scale="1.0 1.0 1.0" /> -->
+        <mesh filename="file://$(find xarm_description)/meshes/link3_collision.stl" scale="1.0 1.0 1.0" />
+      </geometry>
+    </collision>
+    <inertial>
+      <mass value="0.1"/>
+      <inertia ixx="0.4" ixy="0.0" ixz="0.0" iyy="0.4" iyz="0.0" izz="0.2"/>
+    </inertial>
+  </link>
+  <joint name="arm2" type="revolute">
+    <limit effort="1000" lower="-1.95" upper="1.95" velocity="1.0" />
+    <parent link="link3"/>
+    <child link="link2"/>
+    <origin rpy="0.0 0.0 0.0" xyz="-0.00125 0.0 0.050"/>
+    <axis xyz="0 0 1"/>
+  </joint>
+  <link name="link2">
+    <visual>
+      <origin rpy="0 0 0" xyz="0.0 0.0 0.0" />
+      <geometry>
+        <!-- <mesh filename="package://xarm_description/meshes/link2.stl" scale="1.0 1.0 1.0" /> -->
+        <mesh filename="file://$(find xarm_description)/meshes/link2.stl" scale="1.0 1.0 1.0" />
+      </geometry>
+      <material name="black" />
+    </visual>
+    <collision>
+      <origin rpy="0 0 0" xyz="0 0 0" />
+      <geometry>
+        <!-- <mesh filename="package://xarm_description/meshes/link2_collision.stl" scale="1.0 1.0 1.0" /> -->
+        <mesh filename="file://$(find xarm_description)/meshes/link2_collision.stl" scale="1.0 1.0 1.0" />
+      </geometry>
+    </collision>
+    <inertial>
+      <mass value="0.1"/>
+      <inertia ixx="0.4" ixy="0.0" ixz="0.0" iyy="0.4" iyz="0.0" izz="0.2"/>
+    </inertial>
+  </link>
+  <joint name="arm1" type="revolute">
+    <limit effort="1000" lower="0" upper="1.8326" velocity="1.0" />
+    <parent link="link2"/>
+    <child link="link1"/>
+    <origin xyz="-0.0015 -0.014 0.0315" rpy="0.0 0.0 0.0" />
+    <axis xyz="1 0 0"/>
+  </joint>
+  <link name="link1">
+    <visual>
+      <origin rpy="0 0 0" xyz="0.0 0.0 0.0" />
+      <geometry>
+        <!-- <mesh filename="package://xarm_description/meshes/link1.stl" scale="1.0 1.0 1.0" /> -->
+        <mesh filename="file://$(find xarm_description)/meshes/link1.stl" scale="1.0 1.0 1.0" />
+      </geometry>
+      <material name="black" />
+    </visual>
+    <collision>
+      <origin rpy="0 0 0" xyz="0 0 0" />
+      <geometry>
+        <!-- <mesh filename="package://xarm_description/meshes/link1_collision.stl" scale="1.0 1.0 1.0" /> -->
+        <mesh filename="file://$(find xarm_description)/meshes/link1_collision.stl" scale="1.0 1.0 1.0" />
+      </geometry>
+    </collision>
+    <inertial>
+      <mass value="0.1"/>
+      <inertia ixx="0.4" ixy="0.0" ixz="0.0" iyy="0.4" iyz="0.0" izz="0.2"/>
+    </inertial>
+  </link>
+  <joint name="arm1_left" type="continuous">
+    <parent link="link2"/>
+    <child link="link1_left"/>
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