Commit message: Remove unnecessary files

File: xarm_moveit_config/config/xarm.ros2_control.xacro (robot description, xacro)
@@ -1,130 +1,86 @@
 <?xml version="1.0"?>
 <robot xmlns:xacro="http://www.ros.org/wiki/xacro">
-  <xacro:macro name="xarm_ros2_control" params="name initial_positions_file controllers sim_robot">
-    <xacro:property name="initial_positions"
-      value="${xacro.load_yaml(initial_positions_file)['initial_positions']}" />
-    <xacro:if value="${sim_robot}">
-      <gazebo reference="world">
-      </gazebo>
-      <gazebo>
-        <plugin filename="libgazebo_ros2_control.so" name="gazebo_ros2_control">
-          <parameters>$(arg controllers)</parameters>
-        </plugin>
-      </gazebo>
-      <ros2_control name="GazeboSystem" type="system">
-        <hardware>
-          <!-- By default, set up controllers for simulation. This won't work on real hardware -->
-          <plugin>gazebo_ros2_control/GazeboSystem</plugin>
-        </hardware>
-        <joint name="xarm_6_joint">
-          <command_interface name="position" />
-          <state_interface name="position">
-            <param name="initial_value">${initial_positions['xarm_6_joint']}</param>
-          </state_interface>
-          <state_interface name="velocity" />
-        </joint>
-        <joint name="xarm_5_joint">
-          <command_interface name="position" />
-          <state_interface name="position">
-            <param name="initial_value">${initial_positions['xarm_5_joint']}</param>
-          </state_interface>
-          <state_interface name="velocity" />
-        </joint>
-        <joint name="xarm_4_joint">
-          <command_interface name="position" />
-          <state_interface name="position">
-            <param name="initial_value">${initial_positions['xarm_4_joint']}</param>
-          </state_interface>
-          <state_interface name="velocity" />
-        </joint>
-        <joint name="xarm_3_joint">
-          <command_interface name="position" />
-          <state_interface name="position">
-            <param name="initial_value">${initial_positions['xarm_3_joint']}</param>
-          </state_interface>
-          <state_interface name="velocity" />
-        </joint>
-        <joint name="xarm_2_joint">
-          <command_interface name="position" />
-          <state_interface name="position">
-            <param name="initial_value">${initial_positions['xarm_2_joint']}</param>
-          </state_interface>
-          <state_interface name="velocity" />
-        </joint>
-        <joint name="finger_l_joint">
-          <command_interface name="position" />
-          <state_interface name="position">
-            <param name="initial_value">${initial_positions['finger_l_joint']}</param>
-          </state_interface>
-          <state_interface name="velocity" />
-        </joint>
-        <joint name="finger_r_joint">
-          <command_interface name="position" />
-          <state_interface name="position">
-            <param name="initial_value">${initial_positions['finger_r_joint']}</param>
-          </state_interface>
-          <state_interface name="velocity" />
-        </joint>
-      </ros2_control>
-    </xacro:if>
-    <xacro:unless value="${sim_robot}">
-      <ros2_control name="${name}" type="system">
-        <hardware>
-          <plugin>topic_based_ros2_control/TopicBasedSystem</plugin>
-          <param name="joint_commands_topic">/multi_servo_cmd_sub</param>
-          <param name="joint_states_topic">/servo_pos_publisher</param>
-        </hardware>
-        <joint name="xarm_6_joint">
-          <command_interface name="position" />
-          <state_interface name="position">
-            <param name="initial_value">${initial_positions['xarm_6_joint']}</param>
-          </state_interface>
-          <state_interface name="velocity" />
-        </joint>
-        <joint name="xarm_5_joint">
-          <command_interface name="position" />
-          <state_interface name="position">
-            <param name="initial_value">${initial_positions['xarm_5_joint']}</param>
-          </state_interface>
-          <state_interface name="velocity" />
-        </joint>
-        <joint name="xarm_4_joint">
-          <command_interface name="position" />
-          <state_interface name="position">
-            <param name="initial_value">${initial_positions['xarm_4_joint']}</param>
-          </state_interface>
-          <state_interface name="velocity" />
-        </joint>
-        <joint name="xarm_3_joint">
-          <command_interface name="position" />
-          <state_interface name="position">
-            <param name="initial_value">${initial_positions['xarm_3_joint']}</param>
-          </state_interface>
-          <state_interface name="velocity" />
-        </joint>
-        <joint name="xarm_2_joint">
-          <command_interface name="position" />
-          <state_interface name="position">
-            <param name="initial_value">${initial_positions['xarm_2_joint']}</param>
-          </state_interface>
-          <state_interface name="velocity" />
-        </joint>
-        <joint name="finger_l_joint">
-          <command_interface name="position" />
-          <state_interface name="position">
-            <param name="initial_value">${initial_positions['finger_l_joint']}</param>
-          </state_interface>
-          <state_interface name="velocity" />
-        </joint>
-        <joint name="finger_r_joint">
-          <param name="mimic">finger_l_joint</param>
-          <param name="multiplier">1</param>
-          <state_interface name="position">
-            <param name="initial_value">${initial_positions['finger_r_joint']}</param>
-          </state_interface>
-          <state_interface name="velocity" />
-        </joint>
-      </ros2_control>
-    </xacro:unless>
-  </xacro:macro>
+    <xacro:macro name="xarm_ros2_control" params="name initial_positions_file is_simulation">
+        <xacro:property name="initial_positions" value="${xacro.load_yaml(initial_positions_file)['initial_positions']}"/>
+        <gazebo>
+          <plugin filename="libgz_ros2_control-system.so" name="gz_ros2_control::GazeboSimROS2ControlPlugin">
+            <parameters>$(find xarm_moveit_config)/config/ros2_controllers.yaml</parameters>
+          </plugin>
+        </gazebo>
+        <ros2_control name="${name}" type="system">
+            <hardware>
+                <!-- By default, set up controllers for simulation. This won't work on real hardware -->
+                <xacro:if value="${is_simulation}">
+                  <plugin>gz_ros2_control/GazeboSimSystem</plugin>
+                </xacro:if>
+                <xacro:unless value="${is_simulation}">
+                  <plugin>mock_components/GenericSystem</plugin>
+                </xacro:unless>
+            </hardware>
+            <joint name="arm6">
+                <command_interface name="position">
+                  <param name="min">-2.09439435</param>
+                  <param name="max">2.09439435</param>
+                </command_interface>
+                <state_interface name="position">
+                  <param name="initial_value">${initial_positions['arm6']}</param>
+                </state_interface>
+                <state_interface name="velocity"/>
+            </joint>
+            <joint name="arm5">
+                <command_interface name="position">
+                  <param name="min">-2.09439435</param>
+                  <param name="max">2.09439435</param>
+                </command_interface>
+                <state_interface name="position">
+                  <param name="initial_value">${initial_positions['arm5']}</param>
+                </state_interface>
+                <state_interface name="velocity"/>
+            </joint>
+            <joint name="arm4">
+                <command_interface name="position">
+                  <param name="min">-2.09439435</param>
+                  <param name="max">2.09439435</param>
+                </command_interface>
+                <state_interface name="position">
+                  <param name="initial_value">${initial_positions['arm4']}</param>
+                </state_interface>
+                <state_interface name="velocity"/>
+            </joint>
+            <joint name="arm3">
+                <command_interface name="position">
+                  <param name="min">-2.09439435</param>
+                  <param name="max">2.09439435</param>
+                </command_interface>
+                <state_interface name="position">
+                  <param name="initial_value">${initial_positions['arm3']}</param>
+                </state_interface>
+                <state_interface name="velocity"/>
+            </joint>
+            <joint name="arm2">
+                <command_interface name="position">
+                  <param name="min">-2.09439435</param>
+                  <param name="max">2.09439435</param>
+                </command_interface>
+                <state_interface name="position">
+                  <param name="initial_value">${initial_positions['arm2']}</param>
+                </state_interface>
+                <state_interface name="velocity"/>
+            </joint>
+            <joint name="arm1">
+                <command_interface name="position">
+                  <param name="min">0</param>
+                  <param name="max">0.8464847</param>
+                </command_interface>
+                <state_interface name="position">
+                  <param name="initial_value">${initial_positions['arm1']}</param>
+                </state_interface>
+                <state_interface name="velocity"/>
+            </joint>
+            <joint name="arm1_left">
+                <state_interface name="position"/>
+                <state_interface name="velocity"/>
+            </joint>
+        </ros2_control>
+    </xacro:macro>
 </robot>

File: xarm_moveit_config/config/xarm.urdf.xacro (robot description, xacro)
@@ -2,13 +2,14 @@
 <robot xmlns:xacro="http://www.ros.org/wiki/xacro" name="xarm">
     <xacro:arg name="initial_positions_file" default="initial_positions.yaml" />
-    <xacro:arg name="controllers" default="" />
-    <xacro:arg name="sim_robot" default="false"/>
+    <xacro:arg name="is_simulation" default="false" />
     <!-- Import xarm urdf file -->
-    <xacro:include filename="$(find xarm_description)/urdf/xarm_world.urdf.xacro" />
+    <xacro:include filename="$(find xarm_description)/urdf/xarm.urdf.xacro" />
     <!-- Import control_xacro -->
     <xacro:include filename="xarm.ros2_control.xacro" />
-    <xacro:xarm_ros2_control name="System"
-        initial_positions_file="$(arg initial_positions_file)"
-        controllers="$(arg controllers)"
-        sim_robot="$(arg sim_robot)"/>
+    <xacro:if value="$(arg is_simulation)">
+        <xacro:xarm_ros2_control name="GazeboSimSystem" initial_positions_file="$(arg initial_positions_file)" is_simulation="$(arg is_simulation)"/>
+    </xacro:if>
+    <xacro:unless value="$(arg is_simulation)">
+        <xacro:xarm_ros2_control name="FakeSystem" initial_positions_file="$(arg initial_positions_file)" is_simulation="$(arg is_simulation)"/>
+    </xacro:unless>
 </robot>

Commit message: Fixed gripper positions

File: xarm_description/urdf/xarm.urdf.xacro (robot description, xacro)
@@ -233,7 +233,7 @@
     <parent link="link1"/>
     <child link="link0"/>
-    <origin xyz="-0.0023 0.0 0.0305" rpy="0.0 0.0 0.0" />
+    <origin xyz="-0.0023 0.0 0.0305" rpy="-0.3 0.0 0.0" />
     <axis xyz="1 0 0"/>
-    <mimic joint="arm1" multiplier="-1.01" offset="-0.3" />
+    <mimic joint="arm1" multiplier="-1.01" offset="0.0" />
   </joint>
   <link name="link0">
@@ -261,7 +261,7 @@
     <parent link="link1_left"/>
     <child link="link0_left"/>
-    <origin xyz="-0.0023 0.0 0.0305" rpy="0.0 0.0 0.0" />
+    <origin xyz="-0.0023 0.0 0.0305" rpy="0.3 0.0 0.0" />
     <axis xyz="1 0 0"/>
-    <mimic joint="arm1" multiplier="1.01" offset="0.3" />
+    <mimic joint="arm1" multiplier="1.01" offset="0.0" />
   </joint>
   <link name="link0_left">

File: xarm_moveit_config/config/xarm.ros2_control.xacro (robot description, xacro)
@@ -82,4 +82,16 @@
                 <state_interface name="velocity"/>
             </joint>
+            <joint name="arm0">
+                <state_interface name="position">
+                  <param name="initial_value">-0.3</param>
+                </state_interface>
+                <state_interface name="velocity"/>
+            </joint>
+            <joint name="arm0_left">
+                <state_interface name="position">
+                  <param name="initial_value">0.3</param>
+                </state_interface>
+                <state_interface name="velocity"/>
+            </joint>
         </ros2_control>
     </xacro:macro>
