Commit message: Modified rotation axis to match real robot

File: xarm_description/urdf/xarm.urdf.xacro (robot description, xacro)
@@ -1,15 +1,15 @@
-<?xml version="1.0" ?>
+<?xml version="1.0"?>
 <robot xmlns:xacro="http://www.ros.org/wiki/xacro" name="xarm">
   <material name="black">
-    <color rgba="0.2 0.2 0.2 1"/>
+    <color rgba="0.2 0.2 0.2 1" />
   </material>
   <material name="blue">
-    <color rgba="0.3 0.5 0.9 1.0"/>
+    <color rgba="0.3 0.5 0.9 1.0" />
   </material>
-  <link name="world"/>
+  <link name="world" />
   <joint name="world_joint" type="fixed">
-    <parent link="world"/>
-    <child link="base_link"/>
-    <origin rpy="0.0 0.0 0.0" xyz="0.0 0.0 0.0"/>
+    <parent link="world" />
+    <child link="base_link" />
+    <origin rpy="0.0 0.0 0.0" xyz="0.0 0.0 0.0" />
   </joint>
   <link name="base_link">
@@ -25,19 +25,21 @@
       <origin rpy="0 0 0" xyz="0 0 0" />
       <geometry>
-        <!-- <mesh filename="package://xarm_description/meshes/base_collision.stl" scale="1.0 1.0 1.0" /> -->
-        <mesh filename="file://$(find xarm_description)/meshes/base_collision.stl" scale="1.0 1.0 1.0" />
-      </geometry>
-    </collision>
-    <inertial>
-      <mass value="0.1"/>
-      <inertia ixx="0.4" ixy="0.0" ixz="0.0" iyy="0.4" iyz="0.0" izz="0.2"/>
+        <!-- <mesh filename="package://xarm_description/meshes/base_collision.stl" scale="1.0 1.0
+        1.0" /> -->
+        <mesh filename="file://$(find xarm_description)/meshes/base_collision.stl"
+          scale="1.0 1.0 1.0" />
+      </geometry>
+    </collision>
+    <inertial>
+      <mass value="0.1" />
+      <inertia ixx="0.4" ixy="0.0" ixz="0.0" iyy="0.4" iyz="0.0" izz="0.2" />
     </inertial>
   </link>
   <joint name="arm6" type="revolute">
     <limit effort="1000" lower="-2.1" upper="2.1" velocity="1.0" />
-    <parent link="base_link"/>
-    <child link="link6"/>
-    <origin rpy="0.0 0.0 0.0" xyz="0.0 0.0 0.043"/>
-    <axis xyz="0 0 1"/>
+    <parent link="base_link" />
+    <child link="link6" />
+    <origin rpy="0.0 0.0 0.0" xyz="0.0 0.0 0.043" />
+    <axis xyz="0 0 1" />
   </joint>
   <link name="link6">
@@ -53,19 +55,21 @@
       <origin rpy="0 0 0" xyz="0 0 0" />
       <geometry>
-        <!-- <mesh filename="package://xarm_description/meshes/link6_collision.stl" scale="1.0 1.0 1.0" /> -->
-        <mesh filename="file://$(find xarm_description)/meshes/link6_collision.stl" scale="1.0 1.0 1.0" />
-      </geometry>
-    </collision>
-    <inertial>
-      <mass value="0.1"/>
-      <inertia ixx="0.4" ixy="0.0" ixz="0.0" iyy="0.4" iyz="0.0" izz="0.2"/>
+        <!-- <mesh filename="package://xarm_description/meshes/link6_collision.stl" scale="1.0 1.0
+        1.0" /> -->
+        <mesh filename="file://$(find xarm_description)/meshes/link6_collision.stl"
+          scale="1.0 1.0 1.0" />
+      </geometry>
+    </collision>
+    <inertial>
+      <mass value="0.1" />
+      <inertia ixx="0.4" ixy="0.0" ixz="0.0" iyy="0.4" iyz="0.0" izz="0.2" />
     </inertial>
   </link>
   <joint name="arm5" type="revolute">
     <limit effort="1000" lower="-1.5708" upper="1.5708" velocity="1.0" />
-    <parent link="link6"/>
-    <child link="link5"/>
-    <origin rpy="0.0 0.0 0.0" xyz="0.002 0.0 0.032"/>
-    <axis xyz="0 1 0"/>
+    <parent link="link6" />
+    <child link="link5" />
+    <origin rpy="0.0 0.0 0.0" xyz="0.002 0.0 0.032" />
+    <axis xyz="0 -1 0" />
   </joint>
   <link name="link5">
@@ -81,19 +85,21 @@
       <origin rpy="0 0 0" xyz="0 0 0" />
       <geometry>
-        <!-- <mesh filename="package://xarm_description/meshes/link5_collision.stl" scale="1.0 1.0 1.0" /> -->
-        <mesh filename="file://$(find xarm_description)/meshes/link5_collision.stl" scale="1.0 1.0 1.0" />
-      </geometry>
-    </collision>
-    <inertial>
-      <mass value="0.1"/>
-      <inertia ixx="0.4" ixy="0.0" ixz="0.0" iyy="0.4" iyz="0.0" izz="0.2"/>
+        <!-- <mesh filename="package://xarm_description/meshes/link5_collision.stl" scale="1.0 1.0
+        1.0" /> -->
+        <mesh filename="file://$(find xarm_description)/meshes/link5_collision.stl"
+          scale="1.0 1.0 1.0" />
+      </geometry>
+    </collision>
+    <inertial>
+      <mass value="0.1" />
+      <inertia ixx="0.4" ixy="0.0" ixz="0.0" iyy="0.4" iyz="0.0" izz="0.2" />
     </inertial>
   </link>
   <joint name="arm4" type="revolute">
     <limit effort="1000" lower="-2.09" upper="2.09" velocity="1.0" />
-    <parent link="link5"/>
-    <child link="link4"/>
-    <origin rpy="0.0 0.0 0.0" xyz="0.0 0.0 0.09775"/>
-    <axis xyz="0 1 0"/>
+    <parent link="link5" />
+    <child link="link4" />
+    <origin rpy="0.0 0.0 0.0" xyz="0.0 0.0 0.09775" />
+    <axis xyz="0 1 0" />
   </joint>
   <link name="link4">
@@ -109,19 +115,21 @@
       <origin rpy="0 0 0" xyz="0 0 0" />
       <geometry>
-        <!-- <mesh filename="package://xarm_description/meshes/link4_collision.stl" scale="1.0 1.0 1.0" /> -->
-        <mesh filename="file://$(find xarm_description)/meshes/link4_collision.stl" scale="1.0 1.0 1.0" />
-      </geometry>
-    </collision>
-    <inertial>
-      <mass value="0.1"/>
-      <inertia ixx="0.4" ixy="0.0" ixz="0.0" iyy="0.4" iyz="0.0" izz="0.2"/>
+        <!-- <mesh filename="package://xarm_description/meshes/link4_collision.stl" scale="1.0 1.0
+        1.0" /> -->
+        <mesh filename="file://$(find xarm_description)/meshes/link4_collision.stl"
+          scale="1.0 1.0 1.0" />
+      </geometry>
+    </collision>
+    <inertial>
+      <mass value="0.1" />
+      <inertia ixx="0.4" ixy="0.0" ixz="0.0" iyy="0.4" iyz="0.0" izz="0.2" />
     </inertial>
   </link>
   <joint name="arm3" type="revolute">
     <limit effort="1000" lower="-1.85" upper="2.07" velocity="1.0" />
-    <parent link="link4"/>
-    <child link="link3"/>
-    <origin rpy="0.0 0.0 0.0" xyz="0.0 0.0 0.099"/>
-    <axis xyz="0 1 0"/>
+    <parent link="link4" />
+    <child link="link3" />
+    <origin rpy="0.0 0.0 0.0" xyz="0.0 0.0 0.099" />
+    <axis xyz="0 -1 0" />
   </joint>
   <link name="link3">
@@ -137,19 +145,21 @@
       <origin rpy="0 0 0" xyz="0 0 0" />
       <geometry>
-        <!-- <mesh filename="package://xarm_description/meshes/link3_collision.stl" scale="1.0 1.0 1.0" /> -->
-        <mesh filename="file://$(find xarm_description)/meshes/link3_collision.stl" scale="1.0 1.0 1.0" />
-      </geometry>
-    </collision>
-    <inertial>
-      <mass value="0.1"/>
-      <inertia ixx="0.4" ixy="0.0" ixz="0.0" iyy="0.4" iyz="0.0" izz="0.2"/>
+        <!-- <mesh filename="package://xarm_description/meshes/link3_collision.stl" scale="1.0 1.0
+        1.0" /> -->
+        <mesh filename="file://$(find xarm_description)/meshes/link3_collision.stl"
+          scale="1.0 1.0 1.0" />
+      </geometry>
+    </collision>
+    <inertial>
+      <mass value="0.1" />
+      <inertia ixx="0.4" ixy="0.0" ixz="0.0" iyy="0.4" iyz="0.0" izz="0.2" />
     </inertial>
   </link>
   <joint name="arm2" type="revolute">
     <limit effort="1000" lower="-1.95" upper="1.95" velocity="1.0" />
-    <parent link="link3"/>
-    <child link="link2"/>
-    <origin rpy="0.0 0.0 0.0" xyz="-0.00125 0.0 0.050"/>
-    <axis xyz="0 0 1"/>
+    <parent link="link3" />
+    <child link="link2" />
+    <origin rpy="0.0 0.0 0.0" xyz="-0.00125 0.0 0.050" />
+    <axis xyz="0 0 1" />
   </joint>
   <link name="link2">
@@ -165,19 +175,21 @@
       <origin rpy="0 0 0" xyz="0 0 0" />
       <geometry>
-        <!-- <mesh filename="package://xarm_description/meshes/link2_collision.stl" scale="1.0 1.0 1.0" /> -->
-        <mesh filename="file://$(find xarm_description)/meshes/link2_collision.stl" scale="1.0 1.0 1.0" />
-      </geometry>
-    </collision>
-    <inertial>
-      <mass value="0.1"/>
-      <inertia ixx="0.4" ixy="0.0" ixz="0.0" iyy="0.4" iyz="0.0" izz="0.2"/>
+        <!-- <mesh filename="package://xarm_description/meshes/link2_collision.stl" scale="1.0 1.0
+        1.0" /> -->
+        <mesh filename="file://$(find xarm_description)/meshes/link2_collision.stl"
+          scale="1.0 1.0 1.0" />
+      </geometry>
+    </collision>
+    <inertial>
+      <mass value="0.1" />
+      <inertia ixx="0.4" ixy="0.0" ixz="0.0" iyy="0.4" iyz="0.0" izz="0.2" />
     </inertial>
   </link>
   <joint name="arm1" type="revolute">
     <limit effort="1000" lower="0" upper="1.8326" velocity="1.0" />
-    <parent link="link2"/>
-    <child link="link1"/>
+    <parent link="link2" />
+    <child link="link1" />
     <origin xyz="-0.0015 -0.014 0.0315" rpy="0.0 0.0 0.0" />
-    <axis xyz="1 0 0"/>
+    <axis xyz="1 0 0" />
   </joint>
   <link name="link1">
@@ -193,18 +205,20 @@
       <origin rpy="0 0 0" xyz="0 0 0" />
       <geometry>
-        <!-- <mesh filename="package://xarm_description/meshes/link1_collision.stl" scale="1.0 1.0 1.0" /> -->
-        <mesh filename="file://$(find xarm_description)/meshes/link1_collision.stl" scale="1.0 1.0 1.0" />
-      </geometry>
-    </collision>
-    <inertial>
-      <mass value="0.1"/>
-      <inertia ixx="0.4" ixy="0.0" ixz="0.0" iyy="0.4" iyz="0.0" izz="0.2"/>
+        <!-- <mesh filename="package://xarm_description/meshes/link1_collision.stl" scale="1.0 1.0
+        1.0" /> -->
+        <mesh filename="file://$(find xarm_description)/meshes/link1_collision.stl"
+          scale="1.0 1.0 1.0" />
+      </geometry>
+    </collision>
+    <inertial>
+      <mass value="0.1" />
+      <inertia ixx="0.4" ixy="0.0" ixz="0.0" iyy="0.4" iyz="0.0" izz="0.2" />
     </inertial>
   </link>
   <joint name="arm1_left" type="continuous">
-    <parent link="link2"/>
-    <child link="link1_left"/>
+    <parent link="link2" />
+    <child link="link1_left" />
     <origin xyz="-0.0015 0.014 0.0315" rpy="0.0 0.0 0.0" />
-    <axis xyz="1 0 0"/>
+    <axis xyz="1 0 0" />
     <mimic joint="arm1" multiplier="-1" offset="0" />
   </joint>
@@ -213,5 +227,6 @@
       <origin rpy="0 0 0" xyz="0.0 0.0 0.0" />
       <geometry>
-        <!-- <mesh filename="package://xarm_description/meshes/link1_left.stl" scale="1.0 1.0 1.0" /> -->
+        <!-- <mesh filename="package://xarm_description/meshes/link1_left.stl" scale="1.0 1.0 1.0"
+        /> -->
         <mesh filename="file://$(find xarm_description)/meshes/link1_left.stl" scale="1.0 1.0 1.0" />
       </geometry>
@@ -221,18 +236,20 @@
       <origin rpy="0 0 0" xyz="0 0 0" />
       <geometry>
-        <!-- <mesh filename="package://xarm_description/meshes/link1_left_collision.stl" scale="1.0 1.0 1.0" /> -->
-        <mesh filename="file://$(find xarm_description)/meshes/link1_left_collision.stl" scale="1.0 1.0 1.0" />
-      </geometry>
-    </collision>
-    <inertial>
-      <mass value="0.1"/>
-      <inertia ixx="0.4" ixy="0.0" ixz="0.0" iyy="0.4" iyz="0.0" izz="0.2"/>
+        <!-- <mesh filename="package://xarm_description/meshes/link1_left_collision.stl" scale="1.0
+        1.0 1.0" /> -->
+        <mesh filename="file://$(find xarm_description)/meshes/link1_left_collision.stl"
+          scale="1.0 1.0 1.0" />
+      </geometry>
+    </collision>
+    <inertial>
+      <mass value="0.1" />
+      <inertia ixx="0.4" ixy="0.0" ixz="0.0" iyy="0.4" iyz="0.0" izz="0.2" />
     </inertial>
   </link>
   <joint name="arm0" type="continuous">
-    <parent link="link1"/>
-    <child link="link0"/>
+    <parent link="link1" />
+    <child link="link0" />
     <origin xyz="-0.0023 0.0 0.0305" rpy="-0.3 0.0 0.0" />
-    <axis xyz="1 0 0"/>
+    <axis xyz="1 0 0" />
     <mimic joint="arm1" multiplier="-1.01" offset="0.0" />
   </joint>
@@ -249,18 +266,20 @@
       <origin rpy="0 0 0" xyz="0 0 0" />
       <geometry>
-        <!-- <mesh filename="package://xarm_description/meshes/link0_collision.stl" scale="1.0 1.0 1.0" /> -->
-        <mesh filename="file://$(find xarm_description)/meshes/link0_collision.stl" scale="1.0 1.0 1.0" />
-      </geometry>
-    </collision>
-    <inertial>
-      <mass value="0.1"/>
-      <inertia ixx="0.4" ixy="0.0" ixz="0.0" iyy="0.4" iyz="0.0" izz="0.2"/>
+        <!-- <mesh filename="package://xarm_description/meshes/link0_collision.stl" scale="1.0 1.0
+        1.0" /> -->
+        <mesh filename="file://$(find xarm_description)/meshes/link0_collision.stl"
+          scale="1.0 1.0 1.0" />
+      </geometry>
+    </collision>
+    <inertial>
+      <mass value="0.1" />
+      <inertia ixx="0.4" ixy="0.0" ixz="0.0" iyy="0.4" iyz="0.0" izz="0.2" />
     </inertial>
   </link>
   <joint name="arm0_left" type="continuous">
-    <parent link="link1_left"/>
-    <child link="link0_left"/>
+    <parent link="link1_left" />
+    <child link="link0_left" />
     <origin xyz="-0.0023 0.0 0.0305" rpy="0.3 0.0 0.0" />
-    <axis xyz="1 0 0"/>
+    <axis xyz="1 0 0" />
     <mimic joint="arm1" multiplier="1.01" offset="0.0" />
   </joint>
@@ -269,5 +288,6 @@
       <origin rpy="0 0 0" xyz="0.0 0.0 0.0" />
       <geometry>
-        <!-- <mesh filename="package://xarm_description/meshes/link0_left.stl" scale="1.0 1.0 1.0" /> -->
+        <!-- <mesh filename="package://xarm_description/meshes/link0_left.stl" scale="1.0 1.0 1.0"
+        /> -->
         <mesh filename="file://$(find xarm_description)/meshes/link0_left.stl" scale="1.0 1.0 1.0" />
       </geometry>
@@ -277,11 +297,13 @@
       <origin rpy="0 0 0" xyz="0 0 0" />
       <geometry>
-        <!-- <mesh filename="package://xarm_description/meshes/link0_left_collision.stl" scale="1.0 1.0 1.0" /> -->
-        <mesh filename="file://$(find xarm_description)/meshes/link0_left_collision.stl" scale="1.0 1.0 1.0" />
-      </geometry>
-    </collision>
-    <inertial>
-      <mass value="0.1"/>
-      <inertia ixx="0.4" ixy="0.0" ixz="0.0" iyy="0.4" iyz="0.0" izz="0.2"/>
+        <!-- <mesh filename="package://xarm_description/meshes/link0_left_collision.stl" scale="1.0
+        1.0 1.0" /> -->
+        <mesh filename="file://$(find xarm_description)/meshes/link0_left_collision.stl"
+          scale="1.0 1.0 1.0" />
+      </geometry>
+    </collision>
+    <inertial>
+      <mass value="0.1" />
+      <inertia ixx="0.4" ixy="0.0" ixz="0.0" iyy="0.4" iyz="0.0" izz="0.2" />
     </inertial>
   </link>

Commit message: Added gazebo desk

File: xarm_description/urdf/xarm.urdf.xacro (robot description, xacro)
@@ -11,5 +11,5 @@
     <parent link="world" />
     <child link="base_link" />
-    <origin rpy="0.0 0.0 0.0" xyz="0.0 0.0 0.0" />
+    <origin rpy="0.0 0.0 -1.57" xyz="0.0 0.0 0.0" />
   </joint>
   <link name="base_link">

Commit message: Feat: Improved Gazebo world and added simulated camera

File: xarm_description/urdf/xarm.urdf.xacro (robot description, xacro)
@@ -308,58 +308,5 @@
     </inertial>
   </link>
-  <!-- TO-DO: move out to separate file -->
-  <!-- <joint name="depth_joint" type="fixed">
-    <parent link="link2"/>
-    <child link="depth"/>
-    <origin rpy="-1.5708 0 -1.5708" xyz="0.044 -0.0115 0.045"/>
-  </joint>
-  <link name="depth" /> -->
-  <!-- TO-DO: move out to separate file -->
-  <!-- <ros2_control name="xarm" type="system">
-    <hardware>
-      <plugin>ros2_control_xarm/XArm1SSystemHardware</plugin>
-    </hardware>
-    <joint name="arm6">
-      <command_interface name="position">
-        <param name="min">-2.09439435</param>
-        <param name="max">2.09439435</param>
-      </command_interface>
-      <state_interface name="position"/>
-    </joint>
-    <joint name="arm5">
-      <command_interface name="position">
-        <param name="min">-2.09439435</param>
-        <param name="max">2.09439435</param>
-      </command_interface>
-      <state_interface name="position"/>
-    </joint>
-    <joint name="arm4">
-      <command_interface name="position">
-        <param name="min">-2.09439435</param>
-        <param name="max">2.09439435</param>
-      </command_interface>
-      <state_interface name="position"/>
-    </joint>
-    <joint name="arm3">
-      <command_interface name="position">
-        <param name="min">-2.09439435</param>
-        <param name="max">2.09439435</param>
-      </command_interface>
-      <state_interface name="position"/>
-    </joint>
-    <joint name="arm2">
-      <command_interface name="position">
-        <param name="min">-2.09439435</param>
-        <param name="max">2.09439435</param>
-      </command_interface>
-      <state_interface name="position"/>
-    </joint>
-    <joint name="arm1">
-      <command_interface name="position">
-        <param name="min">0</param>
-        <param name="max">0.8464847</param>
-      </command_interface>
-      <state_interface name="position"/>
-    </joint>
-  </ros2_control> -->
+  <xacro:include filename="camera.urdf.xacro"/>
+  <xacro:camera ref_link="base_link"/>
 </robot>

File: xarm_moveit_config/config/xarm.ros2_control.xacro (robot description, xacro)
@@ -106,4 +106,26 @@
       </xacro:if>
     </ros2_control>
+    <gazebo reference="camera_frame">
+      <sensor name="camera" type="camera">
+        <pose>0 0 0 0 0 0</pose>
+        <visualize>true</visualize>
+        <update_rate>10</update_rate>
+        <camera>
+        <camera_info_topic>camera/camera_info</camera_info_topic>
+          <horizontal_fov>1.089</horizontal_fov>
+          <image>
+            <format>R8G8B8</format>
+            <width>640</width>
+            <height>480</height>
+          </image>
+          <clip>
+            <near>0.05</near>
+            <far>8.0</far>
+          </clip>
+        </camera>
+        <topic>camera/image_raw</topic>
+        <gz_frame_id>camera_frame</gz_frame_id>
+      </sensor>
+    </gazebo>
   </xacro:macro>
 </robot>

Commit message: Updated URDF zero position and simulation params

File: xarm_description/urdf/xarm.urdf.xacro (robot description, xacro)
@@ -37,5 +37,6 @@
   </link>
   <joint name="arm6" type="revolute">
-    <limit effort="1000" lower="-2.1" upper="2.1" velocity="1.0" />
+    <!-- <limit effort="1000" lower="-2.1" upper="2.1" velocity="1.0" /> -->
+    <limit effort="1000" lower="-1.92" upper="1.92" velocity="1.0" />
     <parent link="base_link" />
     <child link="link6" />
@@ -97,5 +98,6 @@
   </link>
   <joint name="arm4" type="revolute">
-    <limit effort="1000" lower="-2.09" upper="2.09" velocity="1.0" />
+    <!-- <limit effort="1000" lower="-2.09" upper="2.09" velocity="1.0" /> -->
+    <limit effort="1000" lower="-1.92" upper="1.92" velocity="1.0" />
     <parent link="link5" />
     <child link="link4" />
@@ -127,5 +129,6 @@
   </link>
   <joint name="arm3" type="revolute">
-    <limit effort="1000" lower="-1.85" upper="2.07" velocity="1.0" />
+    <!-- <limit effort="1000" lower="-1.85" upper="2.07" velocity="1.0" /> -->
+    <limit effort="1000" lower="-1.85" upper="1.85" velocity="1.0" />
     <parent link="link4" />
     <child link="link3" />
@@ -157,5 +160,6 @@
   </link>
   <joint name="arm2" type="revolute">
-    <limit effort="1000" lower="-1.95" upper="1.95" velocity="1.0" />
+    <!-- <limit effort="1000" lower="-1.95" upper="1.95" velocity="1.0" /> -->
+    <limit effort="1000" lower="-1.92" upper="1.92" velocity="1.0" />
     <parent link="link3" />
     <child link="link2" />
@@ -187,5 +191,6 @@
   </link>
   <joint name="arm1" type="revolute">
-    <limit effort="1000" lower="0" upper="1.8326" velocity="1.0" />
+    <!-- <limit effort="1000" lower="0" upper="1.8326" velocity="1.0" /> -->
+    <limit effort="1000" lower="0" upper="0.8464847" velocity="1.0" />
     <parent link="link2" />
     <child link="link1" />

File: xarm_moveit_config/config/xarm.ros2_control.xacro (robot description, xacro)
@@ -21,7 +21,7 @@
           <plugin>xarm_control/XArmSystemHardware</plugin>
           <param name="device">/dev/ttyUSB0</param>
-          <param name="zero_pos">11750 12250 11750 12000 11000 16800</param>
+          <param name="zero_pos">120 120 120 120 110 46</param>
           <param name="baud_rate">230400</param>
-          <param name="timeout_ms">1000</param>
+          <param name="timeout_ms">50</param>
           <param name="reduction">15.0</param>
         </xacro:unless>
@@ -39,6 +39,8 @@
       <joint name="arm5">
         <command_interface name="position">
-          <param name="min">-1.92</param>
-          <param name="max">1.92</param>
+          <!-- <param name="min">-1.92</param> -->
+          <!-- <param name="max">1.92</param> -->
+          <param name="min">-1.5708</param>
+          <param name="max">1.5708</param>
         </command_interface>
         <state_interface name="position">
@@ -59,6 +61,8 @@
       <joint name="arm3">
         <command_interface name="position">
-          <param name="min">-1.92</param>
-          <param name="max">1.92</param>
+          <!-- <param name="min">-1.92</param> -->
+          <!-- <param name="max">1.92</param> -->
+          <param name="min">-1.85</param>
+          <param name="max">1.85</param>
         </command_interface>
         <state_interface name="position">

Commit message: Fixed Gripper joints moveit planning behavior

File: xarm_description/urdf/xarm.urdf.xacro (robot description, xacro)
@@ -192,5 +192,5 @@
   <joint name="arm1" type="revolute">
     <!-- <limit effort="1000" lower="0" upper="1.8326" velocity="1.0" /> -->
-    <limit effort="1000" lower="0" upper="0.8464847" velocity="1.0" />
+    <limit effort="1000" lower="0" upper="2.1118483949" velocity="1.5" />
     <parent link="link2" />
     <child link="link1" />

File: xarm_moveit_config/config/xarm.ros2_control.xacro (robot description, xacro)
@@ -21,5 +21,5 @@
           <plugin>xarm_control/XArmSystemHardware</plugin>
           <param name="device">/dev/ttyUSB0</param>
-          <param name="zero_pos">120 120 120 120 110 46</param>
+          <param name="zero_pos">120 120 120 120 110 170</param>
           <param name="baud_rate">230400</param>
           <param name="timeout_ms">50</param>
